File: portail_jc.kicad_pcb (KiCad board)
At the start: 2 copper layers, 175 x 95 mm, 111 parts, among them J1 Conn_01x02_Male, J10 Conn_01x03_Male, J11 Conn_01x04, J2 Conn_01x04_Male, J3 Conn_01x07_Male, J4 Conn_01x09_Male, J5 Conn_01x03_Male, J6 Screw_Terminal_01x02, J7 Conn_01x04, J8 Conn_01x04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

Commit message: V2.3
Parts:
- removed D3: W04G, Diode_THT:Diode_Bridge_Round_D8.9mm
- removed F3: Fuse, Fuse:Fuseholder_Cylinder-5x20mm_Schurter_0031_8201_Horizontal_Open
- added C11: 100nF, Capacitor_THT:C_Rect_L7.2mm_W2.5mm_P5.00mm_FKS2_FKP2_MKS2_MKP2, F.Cu at (241.6, 107.7)
- added C17: 100nF, Capacitor_THT:C_Rect_L7.2mm_W2.5mm_P5.00mm_FKS2_FKP2_MKS2_MKP2, F.Cu at (238.3, 107.7)
- added C18: 100nF 400V, Capacitor_THT:C_Rect_L16.5mm_W6.0mm_P15.00mm_MKT, F.Cu at (73.8, 118.7)
- added FL1: Wurth 7446223001, Filter:Filtre_wurth, F.Cu at (75.4, 103.6)
- added H14: MountingHole, MountingHole:MountingHole_3.2mm_M3, F.Cu at (152.1, 77.0)
- added H15: MountingHole, MountingHole:MountingHole_3.2mm_M3, F.Cu at (126.7, 68.8)
- added J12: ZMCT103C, Connector_PinSocket_2.54mm:PinSocket_1x04_P2.54mm_Vertical, F.Cu at (152.0, 65.4)
- D1: value 1.5KE300CA -> 1.5KE400CA
- D10, D4: value 1.5KE30CA -> 1.5KE39CA
- D14: value 5.1V -> DZ5.1V
- H11, H12: value MountingHole_Pad -> Pad
- H13: value MountingHole_Pad -> MountingHole; footprint MountingHole:MountingHole_2.2mm_M2_Pad -> MountingHole:MountingHole_3.2mm_M3
- J11, J7, J8: footprint Connector_PinHeader_2.54mm:PinHeader_1x04_P2.54mm_Vertical -> Connector_PinSocket_2.54mm:PinSocket_1x04_P2.54mm_Vertical
- R14: value 1k -> 1,5k
- R2, R27: value 1,2k -> 1,8k
- moved R29 43.8 mm to (94.2, 59.2), turned to 270 degrees
- moved C3 41.2 mm to (100.6, 69.8), turned to 270 degrees
- moved H13 32.8 mm to (152.1, 61.7)
- moved C6 25.3 mm to (106.8, 107.2)
- moved R22 24.8 mm to (103.1, 107.3)
- moved Q5 23.7 mm to (99.3, 82.3)
- moved R19 21.9 mm to (95.8, 99.7)
- moved R20 21.7 mm to (99.4, 107.3)
- moved R7 17.4 mm to (153.0, 109.5), turned to 90 degrees
- moved Q2 16.4 mm to (147.8, 89.8)
- moved C12 15.9 mm to (144.3, 94.6)
- moved C13 15.1 mm to (144.3, 109.6)
- moved Q3 14.9 mm to (147.8, 104.8)
- moved C14 14.8 mm to (144.3, 124.3)
- moved Q4 14.2 mm to (147.8, 119.5)
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Connections:
- net +5V renamed 5V
- net /12VA renamed Net-(D10-Pad1)
- A1 pad 11: Net-(A1-Pad11) -> /BpEch
- A1 pad 26: Net-(A1-Pad26) -> Im_Cour
- A1 pad 6: /BpEch -> Net-(A1-Pad6)
- Bp-Ent1 pad 3: Net-(Bp-Ent1-Pad3) -> GND
- Bp-Ent1 pad 4: Net-(Bp-Ent1-Pad3) -> GND
- BpEch1 pad 3: Net-(BpEch1-Pad3) -> GND
- BpEch1 pad 4: Net-(BpEch1-Pad3) -> GND
- C16 pad 1: Net-(C16-Pad1) -> /24VR
- C2 pad 1: Net-(C16-Pad1) -> /24VR
- C5 pad 1: Ph -> Net-(C5-Pad1)
- C5 pad 2: N -> Net-(C5-Pad2)
- D1 pad 1: N -> Net-(C5-Pad2)
- D1 pad 2: Ph -> Net-(C5-Pad1)
- D12 pad 2: /12VR -> 24V
- D2 pad 1: /12VR -> /24VR
- D5 pad 2: /12VR -> /24VR
- F1 pad 2: Ph -> Net-(C5-Pad1)
- F2 pad 1: /12 -> /24
- J1 pad 2: N -> Net-(C5-Pad2)
- R26 pad 1: Net-(A1-Pad11) -> Net-(A1-Pad6)
- U4 pad 1: Net-(C16-Pad1) -> /24VR
Routing:
- net 5V: track 265.7 -> 348.8 mm
- net /24VR: track 0.00 -> 75.7 mm
- net Net-(C5-Pad2): track 0.00 -> 71.1 mm
- net Im_Cour: track 0.00 -> 65.0 mm
- net Net-(A1-Pad6): track 0.00 -> 57.6 mm, vias 0 -> 1
- net Net-(A1-Pad11): track 50.8 -> 0.00 mm, vias 1 -> 0
- net /12VR: track 40.8 -> 0.00 mm
- net Ph: track 107.2 -> 147.5 mm
- net /12: track 35.6 -> 0.00 mm
- net Net-(C16-Pad1): track 35.2 -> 0.00 mm
- net Net-(C5-Pad1): track 0.00 -> 32.7 mm
- net N: track 135.6 -> 164.4 mm
- net /puissance/U: track 76.7 -> 105.4 mm
- net Net-(C17-Pad1): track 42.7 -> 65.3 mm
- net Net-(H12-Pad1): track 111.8 -> 90.7 mm
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Other:
- net class 1mm added: clearance 0.2, trace_width 1, via_dia 0.8, via_drill 0.4
- board text added: "Arduino NANO V3.0"
- board text added: "Clone de carte CAME BZX6N-7N (C) F1IWQ Sept 2021"
- board text added: "L1T (Ph)"
- board text added: "L2T (N)"
- board text added: "Module Convertisseur ZMCT 103C 5A"
- board text added: "Récepteur télécom."
- board text added: "W (N)"
- board text removed: "Commande portail JC V2.0 F1IWQ Aout 2021"
- board text removed: "L1T"
- board text removed: "L2T"
- board text removed: "Ph (L1T)"
- board text removed: "Récepteur télécommande"
- board text removed: "W"

Commit message: V2.32
Parts:
- removed H11, H12: Pad, MountingHole:MountingHole_2.2mm_M2_Pad
- removed H13, H14, H15: MountingHole, MountingHole:MountingHole_3.2mm_M3
- removed J12: ZMCT103C, Connector_PinSocket_2.54mm:PinSocket_1x04_P2.54mm_Vertical
- added C19: 100nF, Capacitor_THT:C_Rect_L7.2mm_W2.5mm_P5.00mm_FKS2_FKP2_MKS2_MKP2, F.Cu at (224.0, 70.0)
- added C20: 100nF, Capacitor_THT:C_Rect_L7.2mm_W2.5mm_P5.00mm_FKS2_FKP2_MKS2_MKP2, F.Cu at (229.2, 65.3)
- added D3: 1N4004, Diode_THT:D_DO-41_SOD81_P10.16mm_Horizontal, F.Cu at (194.0, 88.5)
- added R40: 220, Resistor_THT:R_Axial_DIN0207_L6.3mm_D2.5mm_P7.62mm_Horizontal, F.Cu at (210.0, 72.5)
- C1: value 1000µF 25V -> 100nF; footprint Capacitor_THT:CP_Radial_D12.5mm_P5.00mm -> Capacitor_THT:C_Rect_L7.2mm_W2.5mm_P5.00mm_FKS2_FKP2_MKS2_MKP2
- R14: value 1,5k -> 220
- R2, R27: value 1,8k -> 4,7k
- R31: value 5,6k -> 6,8k
- R8, R9: value 220 -> 2,7k
- moved C1 25.7 mm to (224.7, 78.0), turned to 270 degrees
- moved C2 2.60 mm to (199.9, 83.0)
Connections:
- net 5V renamed +5V
- A1 pad 26: Im_Cour -> Net-(A1-Pad26)
- C1 pad 1: Net-(C1-Pad1) -> /FC
- C16 pad 1: /24VR -> Net-(C16-Pad1)
- C2 pad 1: /24VR -> Net-(C16-Pad1)
- C9 pad 1: Net-(C1-Pad1) -> Net-(C9-Pad1)
- D12 pad 1: Net-(C1-Pad1) -> Net-(C9-Pad1)
- Q5 pad 2: Net-(H12-Pad1) -> CT
- R1 pad 1: /10 -> Net-(R1-Pad1)
- R22 pad 2: Net-(H12-Pad1) -> CT
- R29 pad 2: Net-(H12-Pad1) -> CT
- R36 pad 1: /10 -> Net-(R1-Pad1)
- U1 pad 1: Net-(C1-Pad1) -> Net-(C9-Pad1)
- U2 pad 1: /10 -> Net-(R1-Pad1)
- U2 pad 7: /10 -> Net-(R1-Pad1)
- U4 pad 1: /24VR -> Net-(C16-Pad1)
Routing:
- net /10: track 203.5 -> 85.2 mm, vias 1 -> 0
- net Net-(R1-Pad1): track 0.00 -> 110.9 mm, vias 0 -> 1
- net Net-(H12-Pad1): track 90.7 -> 0.00 mm
- net CT: track 10.4 -> 91.9 mm
- net Im_Cour: track 65.0 -> 0.00 mm
- net +5V: track 348.8 -> 284.9 mm
- net Net-(C9-Pad1): track 0.00 -> 42.4 mm
- net Net-(C1-Pad1): track 42.4 -> 0.00 mm
- net Net-(C16-Pad1): track 0.00 -> 33.0 mm
- net /24VR: track 75.7 -> 48.0 mm
- net /FC: track 38.5 -> 43.8 mm
- net Net-(R9-Pad1): track 59.6 -> 62.7 mm
- net /F: track 20.2 -> 22.8 mm
- net 24V: track 180.6 -> 183.2 mm
- net Net-(R27-Pad2): track 70.8 -> 68.4 mm
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Other:
- board text added: "Clone V2.0 carte CAME BZX6N-7N (C) F1IWQ Sept 2021"
- board text removed: "Clone de carte CAME BZX6N-7N (C) F1IWQ Sept 2021"
- board text removed: "Module Convertisseur ZMCT 103C 5A"

Commit message: V2.33
Parts:
- removed C11, C17: 100nF, Capacitor_THT:C_Rect_L7.2mm_W2.5mm_P5.00mm_FKS2_FKP2_MKS2_MKP2
Routing:
- net Net-(R24-Pad2): track 65.3 -> 42.7 mm
- net Net-(R3-Pad2): track 41.8 -> 35.8 mm

Commit message: V2.40
Parts:
- moved R40 19.3 mm to (191.1, 68.3)
- moved C16 14.5 mm to (204.0, 88.9), turned to 180 degrees
- moved D12 11.1 mm to (184.2, 83.3), turned to 180 degrees
- moved C2 4.67 mm to (195.3, 82.0)
- moved C15 3.43 mm to (214.4, 76.2)
- moved U4 1.40 mm to (209.3, 85.7)
Routing:
- net Net-(R1-Pad1): track 110.9 -> 131.7 mm
- net /10: track 85.2 -> 66.7 mm
- net Net-(C9-Pad1): track 42.4 -> 52.8 mm
- net Net-(C16-Pad1): track 33.0 -> 26.0 mm
- net Net-(R9-Pad1): track 62.7 -> 58.4 mm
- net Net-(R27-Pad2): track 68.4 -> 66.6 mm
- net /24VR: track 48.0 -> 46.8 mm

Commit message: V2.41
Parts:
- moved R29 0.76 mm to (95.0, 59.2)
- moved D1 0.38 mm to (79.8, 97.0)
- moved C5 0.25 mm to (73.7, 82.0)
Routing:
- net N: track 164.4 -> 174.5 mm
- net CT: track 91.9 -> 81.9 mm
- net /puissance/U: track 105.4 -> 102.4 mm
- net Net-(C5-Pad2): track 71.1 -> 69.4 mm
- net /puissance/V: track 81.5 -> 79.8 mm
- net /puissance/W: track 52.0 -> 52.9 mm

Commit message: 2.43
Parts:
- added REF**: OSHW-Logo2_14.6x12mm_SilkScreen, Symbol:OSHW-Logo2_14.6x12mm_SilkScreen, F.Cu at (99.8, 126.2)
- moved C16 2.63 mm to (201.3, 88.6)
- moved D3 0.96 mm to (193.0, 88.5)
Routing:
- net Net-(A1-Pad7): track 53.4 -> 52.2 mm
- net Net-(C16-Pad1): track 26.0 -> 27.0 mm
- net Net-(C9-Pad1): track 52.8 -> 53.6 mm
- net /24VR: track 46.8 -> 46.3 mm

Commit message: V2.1
Parts:
- removed REF**: OSHW-Logo2_14.6x12mm_SilkScreen, Symbol:OSHW-Logo2_14.6x12mm_SilkScreen
- added FID1: Fiducial, Symbol:KiCad-Logo2_6mm_SilkScreen, F.Cu at (138.7, 60.5)
- added FID2: Fiducial, Symbol:OSHW-Logo2_9.8x8mm_SilkScreen, F.Cu at (100.3, 130.8)
- added R41: 47k, Resistor_THT:R_Axial_DIN0207_L6.3mm_D2.5mm_P7.62mm_Horizontal, F.Cu at (165.1, 119.1)
Routing:
- net /DATA: track 56.3 -> 59.7 mm
Other:
- board text added: "Clone V2.1 carte CAME ZBX6N-7N (C) F1IWQ Sept 2021"
- board text removed: "Clone V2.0 carte CAME BZX6N-7N (C) F1IWQ Sept 2021"
