File: portail_jc.kicad_pcb (KiCad board)
At the start: 2 copper layers, 175 x 95 mm, 115 parts, among them J1 Conn_01x02_Male, J10 Conn_01x03_Male, J11 Conn_01x04, J2 Conn_01x04_Male, J3 Conn_01x07_Male, J4 Conn_01x09_Male, J5 Conn_01x03_Male, J6 Screw_Terminal_01x02, J7 Conn_01x04, J8 Conn_01x04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

Commit message: soft update & schema
Parts:
- R14: value 220 -> 2,7k
Changed lines of the file:
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@@
   (general
     (thickness 1.6)
-    (drawings 64)
+    (drawings 62)
     (tracks 808)
     (zones 0)
@@
       (effects (font (size 1 1) (thickness 0.15)))
     )
-    (fp_text value 220 (at 3.81 2.37 180) (layer F.Fab)
+    (fp_text value 2,7k (at 3.81 2.37 180) (layer F.Fab)
       (effects (font (size 1 1) (thickness 0.15)))
     )
@@
   (gr_line (start 81.026 71.374) (end 84.836 71.374) (layer F.SilkS) (width 0.12))
   (gr_line (start 158.877 59.436) (end 165.354 59.436) (layer F.SilkS) (width 0.12))
-  (gr_line (start 155.829 93.98) (end 162.306 93.98) (layer F.SilkS) (width 0.12))
   (gr_text ENTREE (at 187.325 133.731) (layer F.SilkS)
     (effects (font (size 2 2) (thickness 0.3)))
@@
     (effects (font (size 1 1) (thickness 0.15)))
   )
-  (gr_text 1A-F (at 159.004 92.329) (layer F.SilkS)
+  (gr_text 1A-F (at 154.686 72.644) (layer F.SilkS)
     (effects (font (size 1.2 1.2) (thickness 0.2)))
   )
-  (gr_text 1A-F (at 154.686 80.264) (layer F.SilkS)
-    (effects (font (size 1.2 1.2) (thickness 0.2)))
-  )
-  (gr_text 1A-F (at 162.433 58.42) (layer F.SilkS)
+  (gr_text 1A-F (at 154.686 62.484) (layer F.SilkS)
     (effects (font (size 1.2 1.2) (thickness 0.2)))
   )
