File: portail_jc.sch (KiCad schematic (older format))
At the start: 83 parts, among them J1 Conn_01x02_Male, J10 Conn_01x03_Male, J11 Conn_01x04, J3 Conn_01x07_Male, J4 Conn_01x09_Male, J5 Conn_01x03_Male, J6 Screw_Terminal_01x02, J7 Conn_01x04, J8 Conn_01x04, J9 Conn_01x04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

Commit message: V2.3
Parts:
- removed D3: W04G, Diode_THT:Diode_Bridge_Round_D8.9mm, symbol Diode_Bridge:W04G
- removed F3: Fuse, Fuse:Fuseholder_Cylinder-5x20mm_Schurter_0031_8201_Horizontal_Open, symbol Device:Fuse
- added C11, C17: 100nF, Capacitor_THT:C_Rect_L7.2mm_W2.5mm_P5.00mm_FKS2_FKP2_MKS2_MKP2, symbol Device:C
- added C18: 100nF 400V, Capacitor_THT:C_Rect_L16.5mm_W6.0mm_P15.00mm_MKT, symbol Device:C
- added FL1: Wurth 7446223001, Filter:Filtre_wurth, symbol Device:EMI_Filter_LL
- added H13, H14, H15: MountingHole, MountingHole:MountingHole_3.2mm_M3, symbol Mechanical:MountingHole
- D1: value 1.5KE300CA -> 1.5KE400CA
- D10, D4: value 1.5KE30CA -> 1.5KE39CA
- D14: value 5.1V -> DZ5.1V
- J11, J7, J8: footprint Connector_PinHeader_2.54mm:PinHeader_1x04_P2.54mm_Vertical -> Connector_PinSocket_2.54mm:PinSocket_1x04_P2.54mm_Vertical
- R14: value 1k -> 1,5k
- R2, R27: value 1,2k -> 1,8k
Connections:
- net labels added: 24VR, 5V, Im_Cour
- net labels removed: 12VA, 12VR
- wire segments 306 -> 320
Other:
- note added: "24V Ac"
- note added: "32V PkPk"
- note added: "32V\npkpk"
- note added: "4,7V PkPk"
- note removed: "12V Ac"
- note removed: "C5 optionnel"
- note removed: "max=17V"
- note removed: "max=4,7V"
- moved on the sheet: C1, C15, C16, C2, C4, C5, C9, D1, D12, D9, J9, R17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

Commit message: V2.32
Parts:
- removed C1: 1000µF 25V, Capacitor_THT:CP_Radial_D12.5mm_P5.00mm, symbol Device:CP
- removed H13, H14, H15: MountingHole, MountingHole:MountingHole_3.2mm_M3, symbol Mechanical:MountingHole
- added C1, C19, C20: 100nF, Capacitor_THT:C_Rect_L7.2mm_W2.5mm_P5.00mm_FKS2_FKP2_MKS2_MKP2, symbol Device:C
- added D3: 1N4004, Diode_THT:D_DO-41_SOD81_P10.16mm_Horizontal, symbol Diode:1N4004
- added R40: 220, Resistor_THT:R_Axial_DIN0207_L6.3mm_D2.5mm_P7.62mm_Horizontal, symbol Device:R
- R14: value 1,5k -> 220
- R2, R27: value 1,8k -> 4,7k
- R31: value 5,6k -> 6,8k
- R8, R9: value 220 -> 2,7k
Connections:
- net labels removed: 5V, Im_Cour
- wire segments 320 -> 329
- no-connect marks 15 -> 16
Other:
- note added: "24Vac\n34VPkPk"
- moved on the sheet: C16, C2, D2, F2, R14

Commit message: V2.33
Parts:
- removed C11, C17: 100nF, Capacitor_THT:C_Rect_L7.2mm_W2.5mm_P5.00mm_FKS2_FKP2_MKS2_MKP2, symbol Device:C
Connections:
- wire segments 329 -> 324
Changed lines of the file:
@@
 	7500 3600 7500 3700
-Wire Wire Line
-	7500 2950 7500 3050
 Wire Wire Line
 	7450 4050 7950 4050
@@
 Wire Wire Line
 	7450 5100 7500 5100
-Wire Wire Line
-	7500 5100 7500 5200
 $Comp
 L Device:R R26
@@
 	7950 2350 7950 2300
 Connection ~ 7950 2300
-Wire Wire Line
-	8100 4900 7650 4900
 Wire Wire Line
 	7950 2300 8100 2300
@@
 Wire Wire Line
 	9200 5000 9450 5000
-$Comp
-L Device:C C11
-U 1 1 61322CE0
-P 7650 2900
-F 0 "C11" H 7500 3000 50  0000 L CNN
-F 1 "100nF" H 7550 2700 50  0000 L CNN
-F 2 "Capacitor_THT:C_Rect_L7.2mm_W2.5mm_P5.00mm_FKS2_FKP2_MKS2_MKP2" H 7688 2750 50  0001 C CNN
-F 3 "~" H 7650 2900 50  0001 C CNN
-	1    7650 2900
-	1    0    0    -1
-$EndComp
-Wire Wire Line
-	7650 3050 7500 3050
-Connection ~ 7500 3050
-Wire Wire Line
-	7500 3050 7500 3100
-$Comp
-L Device:C C17
-U 1 1 6133E7ED
-P 7650 5050
-F 0 "C17" H 7800 5050 50  0000 L CNN
-F 1 "100nF" H 7550 4850 50  0000 L CNN
-F 2 "Capacitor_THT:C_Rect_L7.2mm_W2.5mm_P5.00mm_FKS2_FKP2_MKS2_MKP2" H 7688 4900 50  0001 C CNN
-F 3 "~" H 7650 5050 50  0001 C CNN
-	1    7650 5050
-	1    0    0    -1
-$EndComp
-Connection ~ 7650 4900
-Wire Wire Line
-	7650 4900 7450 4900
-Wire Wire Line
-	7650 5200 7500 5200
 Wire Wire Line
 	7450 3400 7800 3400
-Connection ~ 7500 5200
-Wire Wire Line
-	7500 5200 7500 5350
 Wire Notes Line
 	2650 6150 2650 7650
@@
 	9050 2150 9050 2100
 Connection ~ 8750 2150
+Wire Wire Line
+	7500 2950 7500 3100
+Wire Wire Line
+	7450 4900 8100 4900
+Wire Wire Line
+	7500 5100 7500 5350
 $EndSCHEMATC

Commit message: V2.35
Other:
- note removed: "sur la carte d'origine, les 0V des tensions alternatives \nsont reliées au 0V des tensions continues"
Changed lines of the file:
@@
 Text Label 5800 1350 1    50   ~ 0
 1
-Text Notes 3550 2550 0    59   ~ 0
-sur la carte d'origine, les 0V des tensions alternatives \nsont reliées au 0V des tensions continues
 $Comp
 L Connector:Conn_01x03_Male J10

Commit message: V2.40
Other:
- note added: "32V\nPkPk"
- note added: "ACPL-844 ou\n4xSFH620"
- note removed: "32V\npkpk"
- moved on the sheet: C10, C4, C9, D12, D14, D5, D9, R17, R30, R31, R32, U1

Commit message: V2.1
Parts:
- added FID1: Fiducial, Symbol:KiCad-Logo2_6mm_SilkScreen, symbol Mechanical:Fiducial
- added FID2: Fiducial, Symbol:OSHW-Logo2_9.8x8mm_SilkScreen, symbol Mechanical:Fiducial
- added R41: 47k, Resistor_THT:R_Axial_DIN0207_L6.3mm_D2.5mm_P7.62mm_Horizontal, symbol Device:R
Connections:
- wire segments 324 -> 328
Other:
- note removed: "Trous de montage"
- moved on the sheet: C7, J11, J6, J8, J9, R38
Changed lines of the file:
@@
 Sheet 1 2
 Title "Clone de carte CAME BZX6N-7N"
-Date "10/09/2021"
-Rev "2.0"
+Date "30/10/2021"
+Rev "2.1"
 Comp "F1IWQ"
 Comment1 ""
@@
 L Connector:Screw_Terminal_01x02 J6
 U 1 1 611361CB
-P 9550 4700
-F 0 "J6" V 9550 4500 50  0000 R CNN
-F 1 "Screw_Terminal_01x02" V 9550 5650 50  0000 R CNN
-F 2 "TerminalBlock:TerminalBlock_bornier-2_P5.08mm" H 9550 4700 50  0001 C CNN
-F 3 "~" H 9550 4700 50  0001 C CNN
-	1    9550 4700
+P 9550 4600
+F 0 "J6" V 9550 4400 50  0000 R CNN
+F 1 "Screw_Terminal_01x02" V 9550 5550 50  0000 R CNN
+F 2 "TerminalBlock:TerminalBlock_bornier-2_P5.08mm" H 9550 4600 50  0001 C CNN
+F 3 "~" H 9550 4600 50  0001 C CNN
+	1    9550 4600
 	0    1    -1   0
 $EndComp
@@
 L power:GND #PWR02
 U 1 1 611578AD
-P 9550 5150
-F 0 "#PWR02" H 9550 4900 50  0001 C CNN
-F 1 "GND" H 9555 4977 50  0000 C CNN
-F 2 "" H 9550 5150 50  0001 C CNN
-F 3 "" H 9550 5150 50  0001 C CNN
-	1    9550 5150
+P 9550 5050
+F 0 "#PWR02" H 9550 4800 50  0001 C CNN
+F 1 "GND" H 9555 4877 50  0000 C CNN
+F 2 "" H 9550 5050 50  0001 C CNN
+F 3 "" H 9550 5050 50  0001 C CNN
+	1    9550 5050
 	1    0    0    -1
 $EndComp
@@
 Text Notes 7850 800  0    59   ~ 0
 Fins de course
-Text Notes 9500 4600 0    59   ~ 0
+Text Notes 8900 4650 0    59   ~ 0
 Antenne
 $Comp
@@
 Text Notes 9050 2950 0    50   ~ 0
 Fermé
-Text Notes 9900 6400 2    59   ~ 0
+Text Notes 10100 6300 2    59   ~ 0
    Récepteur\ntélécommande\n   433 MHz
-Wire Wire Line
-	9000 5900 9000 6050
 $Comp
 L power:GND #PWR017
 U 1 1 61132DB6
-P 9000 6050
-F 0 "#PWR017" H 9000 5800 50  0001 C CNN
-F 1 "GND" H 9005 5877 50  0000 C CNN
-F 2 "" H 9000 6050 50  0001 C CNN
-F 3 "" H 9000 6050 50  0001 C CNN
-	1    9000 6050
+P 9000 6300
+F 0 "#PWR017" H 9000 6050 50  0001 C CNN
+F 1 "GND" H 9150 6250 50  0000 C CNN
+F 2 "" H 9000 6300 50  0001 C CNN
+F 3 "" H 9000 6300 50  0001 C CNN
+	1    9000 6300
 	1    0    0    -1
 $EndComp
@@
 L power:+5V #PWR016
 U 1 1 6113E36B
-P 9000 5550
-F 0 "#PWR016" H 9000 5400 50  0001 C CNN
-F 1 "+5V" H 9015 5723 50  0000 C CNN
-F 2 "" H 9000 5550 50  0001 C CNN
-F 3 "" H 9000 5550 50  0001 C CNN
-	1    9000 5550
-	1    0    0    -1
-$EndComp
-Wire Wire Line
-	9000 5550 9000 5600
-Text Label 9200 5800 0    50   ~ 0
+P 9000 5450
+F 0 "#PWR016" H 9000 5300 50  0001 C CNN
+F 1 "+5V" H 9015 5623 50  0000 C CNN
+F 2 "" H 9000 5450 50  0001 C CNN
+F 3 "" H 9000 5450 50  0001 C CNN
+	1    9000 5450
+	1    0    0    -1
+$EndComp
+Wire Wire Line
+	9000 5450 9000 5500
+Text Label 9250 5700 0    50   ~ 0
 DATA
 Text Notes 9100 3700 0    50   ~ 0
@@
 Wire Wire Line
 	9600 2550 8900 2550
-Text Notes 9950 6400 0    59   ~ 0
+Text Notes 10250 6300 0    59   ~ 0
 TDCA RX500A\nCHJ-9921\nRXB6
 Wire Wire Line
@@
 L Connector_Generic:Conn_01x01 J9
 U 1 1 6151FF69
-P 9000 5000
-F 0 "J9" H 9080 4992 50  0000 L CNN
-F 1 "Conn_01x04" H 8800 4850 50  0000 L CNN
-F 2 "Connector_PinHeader_2.54mm:PinHeader_1x01_P2.54mm_Vertical" H 9000 5000 50  0001 C CNN
-F 3 "~" H 9000 5000 50  0001 C CNN
-	1    9000 5000
+P 9000 4900
+F 0 "J9" H 9080 4892 50  0000 L CNN
+F 1 "Conn_01x04" H 8800 4750 50  0000 L CNN
+F 2 "Connector_PinHeader_2.54mm:PinHeader_1x01_P2.54mm_Vertical" H 9000 4900 50  0001 C CNN
+F 3 "~" H 9000 4900 50  0001 C CNN
+	1    9000 4900
 	-1   0    0    1
 $EndComp
 Wire Wire Line
-	9450 5000 9450 4900
+	9450 4900 9450 4800
 Wire Wire Line
 	8850 2750 9600 2750
@@
 	1    0    0    -1
 $EndComp
-Text Notes 3250 6500 0    59   ~ 0
-Trous de montage
 Wire Wire Line
 	1750 7100 1600 7100
@@
 L Device:C C7
 U 1 1 611A407B
-P 9000 5750
-F 0 "C7" H 8850 5850 50  0000 L CNN
-F 1 "100nF" H 8750 5650 50  0000 L CNN
-F 2 "Capacitor_THT:C_Rect_L7.2mm_W2.5mm_P5.00mm_FKS2_FKP2_MKS2_MKP2" H 9038 5600 50  0001 C CNN
-F 3 "~" H 9000 5750 50  0001 C CNN
-	1    9000 5750
-	1    0    0    -1
-$EndComp
-Connection ~ 9000 5600
+P 9000 5650
+F 0 "C7" H 8850 5750 50  0000 L CNN
+F 1 "100nF" H 8750 5550 50  0000 L CNN
+F 2 "Capacitor_THT:C_Rect_L7.2mm_W2.5mm_P5.00mm_FKS2_FKP2_MKS2_MKP2" H 9038 5500 50  0001 C CNN
+F 3 "~" H 9000 5650 50  0001 C CNN
+	1    9000 5650
+	1    0    0    -1
+$EndComp
+Connection ~ 9000 5500
 $Comp
 L Device:C C8
@@
 Text GLabel 9750 1600 2    50   Input ~ 0
 24V
-Text Notes 5050 5550 2    50   ~ 0
+Text Notes 5300 5700 2    50   ~ 0
 24V Ac
 Wire Wire Line
@@
 Wire Notes Line
 	2650 6350 4550 6350
-Text Notes 10050 6050 0    50   ~ 0
+Text Notes 10050 5950 0    50   ~ 0
 connecteurs femelle
 $Comp
 L Connector_Generic:Conn_01x04 J8
 U 1 1 6112687D
-P 10700 5800
-F 0 "J8" H 10780 5792 50  0000 L CNN
-F 1 "Conn_01x04" H 10450 5450 50  0000 L CNN
-F 2 "Connector_PinSocket_2.54mm:PinSocket_1x04_P2.54mm_Vertical" H 10700 5800 50  0001 C CNN
-F 3 "~" H 10700 5800 50  0001 C CNN
-	1    10700 5800
+P 10700 5700
+F 0 "J8" H 10780 5692 50  0000 L CNN
+F 1 "Conn_01x04" H 10450 5350 50  0000 L CNN
+F 2 "Connector_PinSocket_2.54mm:PinSocket_1x04_P2.54mm_Vertical" H 10700 5700 50  0001 C CNN
+F 3 "~" H 10700 5700 50  0001 C CNN
+	1    10700 5700
 	1    0    0    1
 $EndComp
@@
 L Device:R R38
 U 1 1 612CC0F5
-P 9700 5800
-F 0 "R38" V 9600 5950 50  0000 C CNN
-F 1 "1,2k" V 9600 5700 50  0000 C CNN
-F 2 "Resistor_THT:R_Axial_DIN0207_L6.3mm_D2.5mm_P7.62mm_Horizontal" V 9630 5800 50  0001 C CNN
-F 3 "~" H 9700 5800 50  0001 C CNN
-	1    9700 5800
+P 9700 5700
+F 0 "R38" V 9600 5850 50  0000 C CNN
+F 1 "1,2k" V 9600 5600 50  0000 C CNN
+F 2 "Resistor_THT:R_Axial_DIN0207_L6.3mm_D2.5mm_P7.62mm_Horizontal" V 9630 5700 50  0001 C CNN
+F 3 "~" H 9700 5700 50  0001 C CNN
+	1    9700 5700
 	0    1    1    0
 $EndComp
 Wire Wire Line
-	9000 5600 10250 5600
+	9000 5500 10250 5500
 Wire Notes Line
 	8700 4450 10950 4450
@@
 L Connector_Generic:Conn_01x04 J11
 U 1 1 612AA2D1
-P 10700 5200
-F 0 "J11" H 10780 5192 50  0000 L CNN
-F 1 "Conn_01x04" H 10450 4850 50  0000 L CNN
-F 2 "Connector_PinSocket_2.54mm:PinSocket_1x04_P2.54mm_Vertical" H 10700 5200 50  0001 C CNN
-F 3 "~" H 10700 5200 50  0001 C CNN
-	1    10700 5200
+P 10700 5100
+F 0 "J11" H 10780 5092 50  0000 L CNN
+F 1 "Conn_01x04" H 10450 4750 50  0000 L CNN
+F 2 "Connector_PinSocket_2.54mm:PinSocket_1x04_P2.54mm_Vertical" H 10700 5100 50  0001 C CNN
+F 3 "~" H 10700 5100 50  0001 C CNN
+	1    10700 5100
 	1    0    0    1
 $EndComp
 Wire Wire Line
-	10500 5300 10250 5300
-Wire Wire Line
-	10250 5300 10250 5600
-Connection ~ 10250 5600
-Wire Wire Line
-	10250 5600 10500 5600
-Wire Wire Line
-	9850 5800 10500 5800
-Wire Wire Line
-	9550 5800 9200 5800
-Connection ~ 9000 5900
-Wire Wire Line
-	9000 5900 10500 5900
-Wire Wire Line
-	10500 5200 10000 5200
+	10500 5200 10250 5200
+Wire Wire Line
+	10250 5200 10250 5500
+Connection ~ 10250 5500
+Wire Wire Line
+	10250 5500 10500 5500
+Wire Wire Line
+	9850 5700 10500 5700
 Wire Wire Line
 	10500 5100 10000 5100
 Wire Wire Line
+	10500 5000 10000 5000
+Wire Wire Line
+	10000 5000 10000 5100
+Wire Wire Line
 	10000 5100 10000 5200
-Wire Wire Line
-	10000 5200 10000 5300
-Connection ~ 10000 5200
+Connection ~ 10000 5100
 $Comp
 L power:GND #PWR020
 U 1 1 6137DFF0
-P 10000 5300
-F 0 "#PWR020" H 10000 5050 50  0001 C CNN
-F 1 "GND" H 10005 5127 50  0000 C CNN
-F 2 "" H 10000 5300 50  0001 C CNN
-F 3 "" H 10000 5300 50  0001 C CNN
-	1    10000 5300
-	1    0    0    -1
-$EndComp
-Connection ~ 9450 5000
-Text Notes 9900 5000 0    50   ~ 0
+P 10000 5200
+F 0 "#PWR020" H 10000 4950 50  0001 C CNN
+F 1 "GND" H 10005 5027 50  0000 C CNN
+F 2 "" H 10000 5200 50  0001 C CNN
+F 3 "" H 10000 5200 50  0001 C CNN
+	1    10000 5200
+	1    0    0    -1
+$EndComp
+Connection ~ 9450 4900
+Text Notes 9900 4900 0    50   ~ 0
 ANT
 Wire Notes Line
@@
 	8700 4450 8700 6450
 Wire Wire Line
-	9450 5000 10500 5000
-Wire Wire Line
-	9550 4900 9550 5150
-Wire Wire Line
-	10500 5700 10150 5700
-NoConn ~ 10150 5700
-Text Label 10250 5700 0    50   ~ 0
+	9450 4900 10500 4900
+Wire Wire Line
+	9550 4800 9550 5050
+Wire Wire Line
+	10500 5600 10150 5600
+NoConn ~ 10150 5600
+Text Label 10250 5600 0    50   ~ 0
 ERR
 Wire Wire Line
@@
 	8900 3150 9600 3150
 Wire Wire Line
-	9200 5000 9450 5000
+	9200 4900 9450 4900
 Wire Wire Line
 	7450 3400 7800 3400
@@
 Text Notes 6900 5350 0    50   ~ 0
 ACPL-844 ou\n4xSFH620
+$Comp
+L Device:R R41
+U 1 1 617EF2DC
+P 9250 6050
+F 0 "R41" H 9100 6050 50  0000 C CNN
+F 1 "47k" H 9100 5950 50  0000 C CNN
+F 2 "Resistor_THT:R_Axial_DIN0207_L6.3mm_D2.5mm_P7.62mm_Horizontal" V 9180 6050 50  0001 C CNN
+F 3 "~" H 9250 6050 50  0001 C CNN
+	1    9250 6050
+	-1   0    0    1
+$EndComp
+Wire Wire Line
+	9250 6250 9000 6250
+Wire Wire Line
+	9000 6250 9000 6300
+Connection ~ 9000 6250
+Wire Wire Line
+	9250 5700 9550 5700
+Wire Wire Line
+	9250 6200 9250 6250
+Wire Wire Line
+	9000 5800 10500 5800
+Wire Wire Line
+	9000 5800 9000 6250
+Connection ~ 9000 5800
+Wire Wire Line
+	9250 5700 9250 5900
+$Comp
+L Mechanical:Fiducial FID1
+U 1 1 617F0846
+P 3000 6500
+F 0 "FID1" H 3085 6546 50  0000 L CNN
+F 1 "Fiducial" H 3085 6455 50  0000 L CNN
+F 2 "Symbol:KiCad-Logo2_6mm_SilkScreen" H 3000 6500 50  0001 C CNN
+F 3 "~" H 3000 6500 50  0001 C CNN
+	1    3000 6500
+	1    0    0    -1
+$EndComp
+$Comp
+L Mechanical:Fiducial FID2
+U 1 1 617F2FD0
+P 3800 6500
+F 0 "FID2" H 3885 6546 50  0000 L CNN
+F 1 "Fiducial" H 3885 6455 50  0000 L CNN
+F 2 "Symbol:OSHW-Logo2_9.8x8mm_SilkScreen" H 3800 6500 50  0001 C CNN
+F 3 "~" H 3800 6500 50  0001 C CNN
+	1    3800 6500
+	1    0    0    -1
+$EndComp
 $EndSCHEMATC

Commit message: soft update & schema
Parts:
- R14: value 220 -> 2,7k
Changed lines of the file:
@@
 encoding utf-8
 Sheet 1 2
-Title "Clone de carte CAME BZX6N-7N"
+Title "Clone de carte CAME ZBX6N-7N"
 Date "30/10/2021"
 Rev "2.1"
@@
 P 9350 1600
 F 0 "R14" V 9557 1600 50  0000 C CNN
-F 1 "220" V 9466 1600 50  0000 C CNN
+F 1 "2,7k" V 9466 1600 50  0000 C CNN
 F 2 "Resistor_THT:R_Axial_DIN0207_L6.3mm_D2.5mm_P7.62mm_Horizontal" V 9280 1600 50  0001 C CNN
 F 3 "~" H 9350 1600 50  0001 C CNN
